File: TAS5760_HAT.sch (KiCad schematic (older format))
At the start: 82 parts, among them J3 40HAT, J9 CONN_01X02, Q1 DMG2305UX, Q2 DMMT5401, U2 CAT24C32

Commit message: 4 flip flops
Design with four flip flops and pll1708
Audio output jumper before filter
Parts:
- removed C? (x2): 10pF, symbol Device:C
- removed C? (x12): C, symbol Device:C
- removed C? (x2): 0.1u, symbol Device:C
- removed C? (x2): 10u, symbol Device:C
- removed C? (x2): 220n, symbol Device:C
- removed C? (x8): 22u, symbol Device:C
- removed C? (x2): 1u, symbol Device:C
- removed J9: CONN_01X02, Connector_PinHeader_2.54mm:PinHeader_1x02_P2.54mm_Vertical, symbol Connector_Generic:Conn_01x02
- removed J?: Screw_Terminal_01x02, symbol Connector:Screw_Terminal_01x02
- removed R11: DNP, Resistor_SMD:R_0603_1608Metric_Pad0.84x1.00mm_HandSolder, symbol Device:R
- removed R?: 24.9K, symbol Device:R
- removed R? (x2): 100K, symbol Device:R
- removed U? (x3): 74HC74, symbol 74xx:74HC74
- added C1, C9: 10u, Capacitor_SMD:C_0603_1608Metric, symbol Device:C_Small
- added C10, C2: 220n, Capacitor_SMD:C_0603_1608Metric, symbol Device:C_Small
- added C11, C23, C25, C26, C3, C31: 1u, Capacitor_SMD:C_0603_1608Metric, symbol Device:C_Small
- added C12, C22, C24, C4, C40, C41, C42, C43, C44: 0u1, Capacitor_SMD:C_0603_1608Metric, symbol Device:C_Small
- added C13, C14, C15, C16, C5, C6: 22u, Capacitor_SMD:C_1206_3216Metric, symbol Device:C_Small
- added C21, C27: 10p, Capacitor_SMD:C_0603_1608Metric, symbol Device:C_Small
- added C32, C33, C34, C35: 0u22, Capacitor_SMD:C_0603_1608Metric, symbol Device:C_Small
- added C36, C37, C38, C39: 0u22, Capacitor_SMD:C_1206_3216Metric, symbol Device:C_Small
- added C45: 470u, Capacitor_SMD:CP_Elec_10x10, symbol Device:CP1_Small
- added D1: LED, LED_SMD:LED_0603_1608Metric, symbol Device:LED
- added F1: Fuse, project_footprints:FuseHolder_OM_Schurter_OMH_125, symbol Device:Fuse
- added H5, H6: 3mm_Mounting_Hole, project_footprints:NPTH_3mm_ID, symbol TAS5760_HAT-rescue:Mounting_Hole-Mechanical
- added J1, J4: SPK_A, TerminalBlock:TerminalBlock_bornier-2_P5.08mm, symbol Connector:Screw_Terminal_01x02
- added JP1, JP2: Jumper_2_Open, project_footprints:Keystone_Jumper_5102, symbol Jumper:Jumper_2_Open
- added L5, L6: L, Inductor_SMD:L_12x12mm_H8mm, symbol Device:L
- added Q3: FDS6890A, Package_SO:SOIC-8_3.9x4.9mm_P1.27mm, symbol Transistor_FET:FDS6890A
- added R10: 24K9, Resistor_SMD:R_0603_1608Metric, symbol Device:R
- added R14, R15: 10K, Resistor_SMD:R_0603_1608Metric, symbol Device:R
- added R3: 4M53, Resistor_SMD:R_0603_1608Metric, symbol Device:R
- added R4: 215K, Resistor_SMD:R_0603_1608Metric, symbol Device:R
- added R5: R, Resistor_SMD:R_0603_1608Metric, symbol Device:R
- added R7: 86K6, Resistor_SMD:R_0603_1608Metric, symbol Device:R
- added U4: LTC4365TS8, Package_TO_SOT_SMD:TSOT-23-8, symbol Power_Management:LTC4365TS8
- added unit 3 of U5
- added unit 3 of U6
- added unit 3 of U7
- C17, C30: renamed from C?; value 10uF -> 10u; footprint (none) -> Capacitor_SMD:C_0603_1608Metric
- C18, C19, C28, C29: renamed from C?; value 0_1uF -> 0u1; footprint (none) -> Capacitor_SMD:C_0603_1608Metric
- C20: renamed from C?; value CP1_Small -> 470u; footprint (none) -> Capacitor_SMD:CP_Elec_10x10
- H1, H2, H3, H4: symbol Mechanical:Mounting_Hole -> TAS5760_HAT-rescue:Mounting_Hole-Mechanical
- J2: renamed from J?; value Screw_Terminal_01x02 -> SPK_A; footprint (none) -> TerminalBlock:TerminalBlock_bornier-2_P5.08mm
- J3: symbol raspberrypi_hat:OX40HAT -> TAS5760_HAT-rescue:OX40HAT-raspberrypi_hat
- L1: renamed from L?; value 6.8u -> 10u; footprint (none) -> Inductor_SMD:L_Bourns_SRN6045TA
- L2: renamed from L?; footprint (none) -> Inductor_SMD:L_Bourns_SRN8040TA
- L3, L4: renamed from L?; footprint (none) -> Inductor_SMD:L_12x12mm_H8mm
- Q1: symbol raspberrypi_hat:DMG2305UX -> TAS5760_HAT-rescue:DMG2305UX-raspberrypi_hat
- Q2: symbol raspberrypi_hat:DMMT5401 -> TAS5760_HAT-rescue:DMMT5401-raspberrypi_hat
- R12, R13: renamed from R?; footprint (none) -> Resistor_SMD:R_0603_1608Metric
- R16: renamed from R?; value R -> 10K; footprint (none) -> Resistor_SMD:R_0603_1608Metric
- R23, R24, R29: footprint Resistor_SMD:R_0603_1608Metric_Pad0.84x1.00mm_HandSolder -> Resistor_SMD:R_0603_1608Metric
- R6, R8: value 3.9K -> 3K9; footprint Resistor_SMD:R_0603_1608Metric_Pad0.84x1.00mm_HandSolder -> Resistor_SMD:R_0603_1608Metric
- R9: renamed from R?; value 43.2K -> 43K2; footprint (none) -> Resistor_SMD:R_0603_1608Metric
- U1: renamed from U?; value LMR33630ADDA -> LMR33610ADDAR; symbol Regulator_Switching:LMR33630ADDA -> Regulator_Switching:LMR33610ADDAR
- U10: renamed from U?; footprint (none) -> TAS5760_HAT:HTSSOP-32_backsolder
- U2: symbol raspberrypi_hat:CAT24C32 -> TAS5760_HAT-rescue:CAT24C32-raspberrypi_hat
- U5, U6, U7, U8: renamed from U?; footprint (none) -> Package_SO:TSSOP-14_4.4x5mm_P0.65mm
- U9: renamed from U?; footprint (none) -> Package_SO:SSOP-20_3.9x8.7mm_P0.635mm
- Y1: renamed from Y?; footprint (none) -> Crystal:Crystal_SMD_SeikoEpson_FA238-4Pin_3.2x2.5mm; symbol Device:Crystal -> Device:Crystal_GND24
- gave numbers to parts that had none: 1
Connections:
- net labels added: BITCLK, DCDC_en, LRCLK, WP, ~SPK_FAULT, ~SPK_SD
- net labels removed: BITCLOCK, ID_SC_EEPROM_pu, ID_SD_EEPROM_pu, LRCK, P3_3V, PG_3_3V, PG_5V
- wire segments 427 -> 512
- no-connect marks 8 -> 31
Other:
- note added: "3V3 DCDC"
- note added: "5V DCDC"
- note added: "Configured to accept 8-28V\n"
- note added: "Derives BIT-clock and Left/Right-clock for i2s from MCLK"
- note added: "Generates MCLK for TAS5760M"
- note added: "I2S clock divider"
- note added: "Input voltage protection"
- note added: "PLL1708 clock generator"
- note added: "Pull WP low to write"
- note added: "TAS5760M amplifier"
- note added: "This is the recommended 5V rail protection for \na HAT with power going to the Pi. See\nhttps://github.com/raspberrypi/hats/blob/master/designguide.md#\nback-powering-the-pi-via-the-j8-gpio-header"
- note removed: "EEPROM WRITE ENABLE"
- note removed: "HAT spec indicates to NEVER\npower the 3.3V pins on the Raspberry Pi \nfrom the HAT header. Only connect the 3.3V\npower from the Pi if the HAT does not have\n3.3V on board.\n\nIF you are designing a board that could\neither be powered by the Pi or from the HAT\nthe jumpers here can be used.\n\nIn most cases, either design the HAT \nto provide the 5V to the Pi and use the\nprotection circuit abov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"
- note removed: "Pullup Resistors"
- note removed: "The HAT spec requires this EEPROM with system information\nto be in place in order to be called a HAT. It should be set up as write\nprotected (WP pin held high), so it may be desirable to either put a \njumper as shown to enable writing, or to hook up a spare IO pin to do so."
- note removed: "These are just pullup resistors for the I2C bus on the EEPROM.\nThe resistor values are per the HAT spec."
- note removed: "This is the recommended 5V rail protection for \na HAT with power going to the Pi.\nSee https://github.com/raspberrypi/hats/blob/master/designguide.md#back-powering-the-pi-via-the-j8-gpio-header"
- moved on the sheet: C17, C18, C19, C20, C28, C29, C30, J2, L3, L4, R12, R13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

Commit message: Updated clock circuit to WM8804
Added optional toslink input and output since wm8804 has digital
input and output. Removed old clock dividing circuit since not needed
since wm8804 has this for free
Parts:
- removed C17, C30: 10u, Capacitor_SMD:C_0603_1608Metric, symbol Device:C_Small
- removed C18, C19, C29, C40, C41, C42, C43: 0u1, Capacitor_SMD:C_0603_1608Metric, symbol Device:C_Small
- removed U5, U6, U7, U8: 74HC74, Package_SO:TSSOP-14_4.4x5mm_P0.65mm, symbol 74xx:74HC74
- removed U9: PLL1708, Package_SO:SSOP-20_3.9x8.7mm_P0.635mm, symbol TAS5760_HAT_2:PLL1708
- added C20, C23, C33, C38, C39: 0u1, Capacitor_SMD:C_0603_1608Metric, symbol Device:C_Small
- added J4: TORX1950, TAS5760_HAT:TORX1950, symbol TAS5760_HAT_2:TORX1950
- added J5: TOTX1950, TAS5760_HAT:TOTX1950, symbol TAS5760_HAT_2:TOTX1950
- added L7: 47u, Inductor_SMD:L_0805_2012Metric, symbol Device:L
- added R12, R13: 100K, Resistor_SMD:R_0603_1608Metric, symbol Device:R
- added R14: 5K6, Resistor_SMD:R_0603_1608Metric, symbol Device:R
- added U4: WM8804, TAS5760_HAT:SSOP-20_5.3x7.2mm_P0.65mm, symbol TAS5760_HAT_2:WM8804
- added U6, U7: 74AHC1G125, TAS5760_HAT:TSSOP-5, symbol TAS5760_HAT:74AHC1G125
- C1: footprint Capacitor_SMD:C_0603_1608Metric -> Capacitor_SMD:C_1206_3216Metric
- C2: renamed from C9; footprint Capacitor_SMD:C_0603_1608Metric -> Capacitor_SMD:C_1206_3216Metric
- L1: renamed from L2; symbol pspice:INDUCTOR -> Device:L
- L2: renamed from L1; symbol pspice:INDUCTOR -> Device:L
- R16: renamed from R23; value 22 -> 10K
- R17: renamed from R24; value 22 -> 47K
- R18: renamed from R6; value 3K9 -> 5K6
- R19: renamed from R8; value 3K9 -> 5K6
- R3: renamed from R5; value R -> 100K
- renumbered C5 to C10, C14 to C11, C6 to C12, C15 to C13, C16 to C14, C45 to C15, C20 to C16, C21 to C17, C44 to C18, C22 to C19, C23 to C21, C27 to C22, C31 to C27, C32 to C29, C2 to C3, C33 to C30, C34 to C31, C35 to C32, C36 to C34, C37 to C35, C38 to C36, C39 to C37, C10 to C4, C3 to C5, C11 to C6, C4 to C7, C12 to C8, C13 to C9, H3 to H2, H2 to H3, J4 to J2, J2 to J3, J3 to J6, Q3 to Q1, Q1 to Q3, R3 to R1, R15 to R10, R16 to R11, R29 to R15, R4 to R2, R7 to R4, R10 to R5, R9 to R6, R13 to R7, R12 to R8, R14 to R9, U3 to U2, U4 to U3, U10 to U5, U2 to U8
Connections:
- net labels added: DATA_IN, MISO
- wire segments 512 -> 431
- no-connect marks 31 -> 18
Other:
- note added: "Changed from 3K9 to 5K6 to reduce part count"
- note removed: "BITCLOCK/256"
- note removed: "Derives BIT-clock and Left/Right-clock for i2s from MCLK"
- note removed: "Generates MCLK for TAS5760M"
- note removed: "I2S clock divider"
- note removed: "MCLK/128"
- note removed: "MCLK/16\n"
- note removed: "MCLK/2"
- note removed: "MCLK/32"
- note removed: "MCLK/4"
- note removed: "MCLK/64"
- note removed: "MCLK/8"
- note removed: "PLL1708 clock generator"
- moved on the sheet: C11, C13, C14, C17, C22, C9, R5, R7, Y1
